File: BaseBoard/Motor.sch (KiCad schematic (older format))
At the start: 14 parts, among them J10 MOTOR, J4 MOTOR, J7 MOTOR, J8 MOTOR, U4 TB6612FNG, U5 TB6612FNG

Commit message: v2提交
Parts:
- C12, C14, C16, C18: footprint Capacitor_SMD:C_0805_2012Metric -> Capacitor_SMD:C_0402_1005Metric
Changed lines of the file:
@@
 F 0 "C14" H 4192 2896 50  0000 L CNN
 F 1 "100nF" H 4192 2805 50  0000 L CNN
-F 2 "Capacitor_SMD:C_0805_2012Metric" H 4100 2850 50  0001 C CNN
+F 2 "Capacitor_SMD:C_0402_1005Metric" H 4100 2850 50  0001 C CNN
 F 3 "~" H 4100 2850 50  0001 C CNN
 	1    4100 2850
@@
 F 0 "C18" H 7792 2896 50  0000 L CNN
 F 1 "100nF" H 7792 2805 50  0000 L CNN
-F 2 "Capacitor_SMD:C_0805_2012Metric" H 7700 2850 50  0001 C CNN
+F 2 "Capacitor_SMD:C_0402_1005Metric" H 7700 2850 50  0001 C CNN
 F 3 "~" H 7700 2850 50  0001 C CNN
 	1    7700 2850
@@
 F 0 "C12" H 2342 2896 50  0000 L CNN
 F 1 "100nF" H 2342 2805 50  0000 L CNN
-F 2 "Capacitor_SMD:C_0805_2012Metric" H 2250 2850 50  0001 C CNN
+F 2 "Capacitor_SMD:C_0402_1005Metric" H 2250 2850 50  0001 C CNN
 F 3 "~" H 2250 2850 50  0001 C CNN
 	1    2250 2850
@@
 F 0 "C16" H 5942 2896 50  0000 L CNN
 F 1 "100nF" H 5942 2805 50  0000 L CNN
-F 2 "Capacitor_SMD:C_0805_2012Metric" H 5850 2850 50  0001 C CNN
+F 2 "Capacitor_SMD:C_0402_1005Metric" H 5850 2850 50  0001 C CNN
 F 3 "~" H 5850 2850 50  0001 C CNN
 	1    5850 2850
