File: BaseBoard/BaseBoard.sch (KiCad schematic (older format))
At the start: 34 parts, among them J1 Raspberry_Pi_2_3, J10 Conn_01x01, J11 Conn_01x01, J12 Conn_01x02_Female, J13 Conn_01x02_Female, J14 Conn_01x02_Female, J15 Conn_01x02_Female, J16 Conn_01x02_Female, J17 MOTOR, J18 MOTOR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

Commit message: 添加BOM，板子上添加IMU接口
Parts:
- added J23: IMU, Connector_PinSocket_2.54mm:PinSocket_1x08_P2.54mm_Vertical, symbol Connector_Generic:Conn_01x08
- U1: symbol custom:SY6912 -> BaseBoard-rescue:SY6912-custom
Connections:
- net labels added: GPIO22, GPIO23, GPIO24, GPIO25, SCL, SDA
Other:
- note added: "VCC\nGND\nSCL\nSDA\nUNO0\nUNO1\nUNO2\nUNO3"
Changed lines of the file:
@@
 $EndComp
 $Comp
-L custom:SY6912 U1
+L BaseBoard-rescue:SY6912-custom U1
 U 1 1 60EA3AD5
 P 8750 5450
@@
 Text Label 7650 2150 2    50   ~ 0
 VBAT
+Text Notes 3000 5550 0    62   ~ 0
+VCC\nGND\nSCL\nSDA\nUNO0\nUNO1\nUNO2\nUNO3
+$Comp
+L Connector_Generic:Conn_01x08 J23
+U 1 1 60EDCB6E
+P 2850 5100
+F 0 "J23" H 2930 5092 50  0000 L CNN
+F 1 "IMU" H 2930 5001 50  0000 L CNN
+F 2 "Connector_PinSocket_2.54mm:PinSocket_1x08_P2.54mm_Vertical" H 2850 5100 50  0001 C CNN
+F 3 "~" H 2850 5100 50  0001 C CNN
+	1    2850 5100
+	1    0    0    -1
+$EndComp
+$Comp
+L power:GND #PWR0161
+U 1 1 60EE0768
+P 2650 4900
+F 0 "#PWR0161" H 2650 4650 50  0001 C CNN
+F 1 "GND" V 2655 4772 50  0000 R CNN
+F 2 "" H 2650 4900 50  0001 C CNN
+F 3 "" H 2650 4900 50  0001 C CNN
+	1    2650 4900
+	0    1    1    0
+$EndComp
+$Comp
+L power:+3.3VA #PWR0162
+U 1 1 60EE0BA2
+P 2650 4800
+F 0 "#PWR0162" H 2650 4650 50  0001 C CNN
+F 1 "+3.3VA" H 2665 4973 50  0000 C CNN
+F 2 "" H 2650 4800 50  0001 C CNN
+F 3 "" H 2650 4800 50  0001 C CNN
+	1    2650 4800
+	0    -1   -1   0
+$EndComp
+Text Label 2950 2000 0    50   ~ 0
+SCL
+Text Label 2950 1900 0    50   ~ 0
+SDA
+Text Label 2650 5100 2    50   ~ 0
+SDA
+Text Label 2650 5000 2    50   ~ 0
+SCL
+Text Label 1350 2700 2    50   ~ 0
+GPIO22
+Text Label 1350 2800 2    50   ~ 0
+GPIO23
+Text Label 1350 2900 2    50   ~ 0
+GPIO24
+Text Label 1350 3000 2    50   ~ 0
+GPIO25
+Text Label 2650 5200 2    50   ~ 0
+GPIO22
+Text Label 2650 5300 2    50   ~ 0
+GPIO23
+Text Label 2650 5400 2    50   ~ 0
+GPIO24
+Text Label 2650 5500 2    50   ~ 0
+GPIO25
 $EndSCHEMATC

Commit message: 更新线路板布局
Parts:
- J12, J13, J16: footprint Connector_PinSocket_2.54mm:PinSocket_1x02_P2.54mm_Vertical -> Connector_Molex:Molex_Mini-Fit_Jr_5566-02A_2x01_P4.20mm_Vertical
- J14: footprint Connector_AMASS:AMASS_XT30U-M_1x02_P5.0mm_Vertical -> Connector_AMASS:AMASS_XT60-M_1x02_P7.20mm_Vertical
Changed lines of the file:
@@
-$EndComp
-$Comp
-L Connector:Conn_01x02_Female J14
-U 1 1 60E8B7DD
-P 7850 2500
-F 0 "J14" H 7878 2476 50  0000 L CNN
-F 1 "Conn_01x02_Female" H 7878 2385 50  0000 L CNN
-F 2 "Connector_AMASS:AMASS_XT30U-M_1x02_P5.0mm_Vertical" H 7850 2500 50  0001 C CNN
-F 3 "~" H 7850 2500 50  0001 C CNN
-	1    7850 2500
-	1    0    0    -1
 $EndComp
 $Comp
@@
 F 0 "J12" H 7878 1576 50  0000 L CNN
 F 1 "Conn_01x02_Female" H 7878 1485 50  0000 L CNN
-F 2 "Connector_PinSocket_2.54mm:PinSocket_1x02_P2.54mm_Vertical" H 7850 1600 50  0001 C CNN
+F 2 "Connector_Molex:Molex_Mini-Fit_Jr_5566-02A_2x01_P4.20mm_Vertical" H 7850 1600 50  0001 C CNN
 F 3 "~" H 7850 1600 50  0001 C CNN
 	1    7850 1600
@@
 F 0 "J13" H 7878 2026 50  0000 L CNN
 F 1 "Conn_01x02_Female" H 7878 1935 50  0000 L CNN
-F 2 "Connector_PinSocket_2.54mm:PinSocket_1x02_P2.54mm_Vertical" H 7850 2050 50  0001 C CNN
+F 2 "Connector_Molex:Molex_Mini-Fit_Jr_5566-02A_2x01_P4.20mm_Vertical" H 7850 2050 50  0001 C CNN
 F 3 "~" H 7850 2050 50  0001 C CNN
 	1    7850 2050
@@
 F 0 "J16" H 7878 3526 50  0000 L CNN
 F 1 "Conn_01x02_Female" H 7878 3435 50  0000 L CNN
-F 2 "Connector_PinSocket_2.54mm:PinSocket_1x02_P2.54mm_Vertical" H 7850 3550 50  0001 C CNN
+F 2 "Connector_Molex:Molex_Mini-Fit_Jr_5566-02A_2x01_P4.20mm_Vertical" H 7850 3550 50  0001 C CNN
 F 3 "~" H 7850 3550 50  0001 C CNN
 	1    7850 3550
@@
 Text Label 2650 5500 2    50   ~ 0
 GPIO25
+$Comp
+L Connector:Conn_01x02_Female J14
+U 1 1 60E8B7DD
+P 7850 2500
+F 0 "J14" H 7878 2476 50  0000 L CNN
+F 1 "Conn_01x02_Female" H 7878 2385 50  0000 L CNN
+F 2 "Connector_AMASS:AMASS_XT60-M_1x02_P7.20mm_Vertical" H 7850 2500 50  0001 C CNN
+F 3 "~" H 7850 2500 50  0001 C CNN
+	1    7850 2500
+	1    0    0    -1
+$EndComp
 $EndSCHEMATC

Commit message: 更新线路板设计，添加PD芯片
Parts:
- removed J15: Conn_01x02_Female, Connector_BarrelJack:BarrelJack_Wuerth_6941xx301002, symbol Connector:Barrel_Jack_Switch
- added C4: 1uF, Capacitor_SMD:C_0805_2012Metric, symbol Device:C_Small
- added D3: SS34, Diode_SMD:D_SMA, symbol Device:D_Shockley
- added J15: USB_C_Receptacle_USB2.0, Connector_USB:USB_C_Receptacle_HRO_TYPE-C-31-M-12, symbol Connector:USB_C_Receptacle_USB2.0
- added R5, R7: 10k, Resistor_SMD:R_0805_2012Metric, symbol Device:R_Small
- added R6: 56k, Resistor_SMD:R_0805_2012Metric, symbol Device:R_Small
- added U2: CH224K, Custom:ESSOP10, symbol Custom:CH224K
- C3: value 10u/X7R -> 10uF/X7R
- J10, J11, J21, J22: footprint TestPoint:TestPoint_Pad_2.0x2.0mm -> Connector_PinHeader_2.54mm:PinHeader_1x01_P2.54mm_Vertical
- J17, J18, J19, J20: footprint Connector_JST:JST_XH_B6B-XH-A_1x06_P2.50mm_Vertical -> Connector_JST:JST_PH_B6B-PH-K_1x06_P2.00mm_Vertical
Connections:
- net labels added: CC1, CC2, DM, DP, VBCHG, VCHARGE
- wire segments 29 -> 37
- no-connect marks 11 -> 16
Other:
- note added: "MOTOR-\nMOTOR+\nENC_A\nENC_VCC\nENC_B\nENC_GND"
- note removed: "CHARGE_PD"
- note removed: "MOTOR-\nENC_VCC\nENC_A\nENC_B\nENC_GND\nMOTOR+"

Commit message: 修正一处电阻阻值错误的问题
Parts:
- R5: value 10k -> 1k
Changed lines of the file:
@@
 P 2000 6100
 F 0 "R5" V 1804 6100 50  0000 C CNN
-F 1 "10k" V 1895 6100 50  0000 C CNN
+F 1 "1k" V 1895 6100 50  0000 C CNN
 F 2 "Resistor_SMD:R_0805_2012Metric" H 2000 6100 50  0001 C CNN
 F 3 "~" H 2000 6100 50  0001 C CNN

Commit message: v2板临时提交
Parts:
- removed C1, C3: 10uF/X7R, Capacitor_SMD:C_0805_2012Metric, symbol Device:C_Small
- removed C2: 470nF, Capacitor_SMD:C_0805_2012Metric, symbol Device:C_Small
- removed C4: 1uF, Capacitor_SMD:C_0805_2012Metric, symbol Device:C_Small
- removed D1: LED_Red, LED_SMD:LED_0805_2012Metric, symbol Device:LED
- removed D2: LED_Green, LED_SMD:LED_0805_2012Metric, symbol Device:LED
- removed D3: SS34, Diode_SMD:D_SMA, symbol Device:D_Shockley
- removed J10, J11, J21, J22: Conn_01x01, Connector_PinHeader_2.54mm:PinHeader_1x01_P2.54mm_Vertical, symbol Connector_Generic:Conn_01x01
- removed J12, J13, J16: Conn_01x02_Female, Connector_Molex:Molex_Mini-Fit_Jr_5566-02A_2x01_P4.20mm_Vertical, symbol Connector:Conn_01x02_Female
- removed J14: Conn_01x02_Female, Connector_AMASS:AMASS_XT60-M_1x02_P7.20mm_Vertical, symbol Connector:Conn_01x02_Female
- removed J15: USB_C_Receptacle_USB2.0, Connector_USB:USB_C_Receptacle_HRO_TYPE-C-31-M-12, symbol Connector:USB_C_Receptacle_USB2.0
- removed J17, J18, J19, J20: MOTOR, Connector_JST:JST_PH_B6B-PH-K_1x06_P2.00mm_Vertical, symbol Connector:Conn_01x06_Female
- removed J2: Longan_A, Connector_PinSocket_2.54mm:PinSocket_1x18_P2.54mm_Vertical, symbol Connector_Generic:Conn_01x18
- removed J3, J4: TB6612_A, Connector_PinSocket_2.54mm:PinSocket_1x08_P2.54mm_Vertical, symbol Connector_Generic:Conn_01x08
- removed J5: Longan_C, Connector_PinSocket_2.54mm:PinSocket_2x04_P2.54mm_Vertical, symbol Connector_Generic:Conn_02x04_Odd_Even
- removed J6: Longan_B, Connector_PinSocket_2.54mm:PinSocket_1x18_P2.54mm_Vertical, symbol Connector_Generic:Conn_01x18
- removed J7, J8: TB6612_B, Connector_PinSocket_2.54mm:PinSocket_1x08_P2.54mm_Vertical, symbol Connector_Generic:Conn_01x08
- removed JP1: SolderJumper_3_Open, Jumper:SolderJumper-3_P1.3mm_Open_Pad1.0x1.5mm_NumberLabels, symbol Jumper:SolderJumper_3_Open
- removed L1: 2.2uH, Inductor_SMD:L_7.3x7.3_H4.5, symbol Device:L
- removed R1: 25mR, Resistor_SMD:R_1206_3216Metric, symbol Device:R_Small
- removed R2, R3, R4, R7: 10k, Resistor_SMD:R_0805_2012Metric, symbol Device:R_Small
- removed R5: 1k, Resistor_SMD:R_0805_2012Metric, symbol Device:R_Small
- removed R6: 56k, Resistor_SMD:R_0805_2012Metric, symbol Device:R_Small
- removed U1: SY6912, Package_SO:HSOP-8-1EP_3.9x4.9mm_P1.27mm_EP2.41x3.1mm_ThermalVias, symbol BaseBoard-rescue:SY6912-custom
- removed U2: CH224K, Custom:ESSOP10, symbol Custom:CH224K
- added C19, C20, C21, C22: 6pF, Capacitor_SMD:C_0603_1608Metric, symbol Device:C_Small
- added C23, C24, C25, C26, C27, C28: 100nF, Capacitor_SMD:C_0805_2012Metric, symbol Device:C_Small
- added D5: LED_Red, LED_SMD:LED_0805_2012Metric, symbol Device:LED
- added J2: USB_C_Receptacle_USB2.0, Connector_USB:USB_C_Receptacle_HRO_TYPE-C-31-M-12, symbol Connector:USB_C_Receptacle_USB2.0
- added J3: Conn_01x04, Connector_JST:JST_PH_B4B-PH-K_1x04_P2.00mm_Vertical, symbol Connector_Generic:Conn_01x04
- added R12: 5.1k, Resistor_SMD:R_0805_2012Metric, symbol Device:R_Small
- added R13, R14: 22R, Resistor_SMD:R_0805_2012Metric, symbol Device:R_Small
- added R15, R16, R19, R20: 10k, Resistor_SMD:R_0805_2012Metric, symbol Device:R_Small
- added R17, R18: 0, Resistor_SMD:R_0805_2012Metric, symbol Device:R_Small
- added SW1, SW2: SW_Push, Button_Switch_SMD:SW_SPST_TL3342, symbol Switch:SW_Push
- added U6: GD32VF103Cx, Package_QFP:LQFP-48_7x7mm_P0.5mm, symbol GD32VF103:GD32VF103Cx
- added Y1: 32.768k, Crystal:Crystal_C38-LF_D3.0mm_L8.0mm_Horizontal, symbol Device:Crystal
- added Y2: 8Mhz, Crystal:Crystal_SMD_5032-2Pin_5.0x3.2mm, symbol Device:Crystal
Connections:
- net labels added: +5VA, BOOT0, BOOT1, LIDAR_RX, LIDAR_TX, OSC32_IN, OSC32_OUT, OSCIN, OSCOUT, USB_DM, USB_DP, VDDA, VSSA
- net labels removed: +12V, CC1, CC2, DM, DP, MOT1_N, MOT1_P, MOT2_N, MOT2_P, MOT3_N, MOT3_P, MOT4_N, MOT4_P, RS, VBAT, VBCHG, VBUS, VCHARGE
- wire segments 37 -> 40
- no-connect marks 16 -> 7
Other:
- note added: "IMU\n"
- note added: "Lidar\n"
- note removed: "5V\n3V3\nB12\nB13\nB14\nB15\nA8\nA11\nA12\nNC\nB4\nB5\nB6\nB7\nB8\nB9\nGND\nGND"
- note removed: "BATTERY CHARGER"
- note removed: "BATT_IN"
- note removed: "C(nF) = 0.02 * T(s)"
- note removed: "CEL"
- note removed: "CHARGE_DC"
- note removed: "DC-DC converter"
- note removed: "EMERGENCY"
- note removed: "GND\nPA9\nPA10\nVCC"
- note removed: "I = 25/R"
- note removed: "JTDO/PB3\nJTDI/PA15\nJTCK/PA14\nJTMS/PA13"
- note removed: "MOTOR CONNECTOR"
- note removed: "MOTOR-\nMOTOR+\nENC_A\nENC_VCC\nENC_B\nENC_GND"
- note removed: "MOTOR1"
- note removed: "MOTOR2"
- note removed: "MOTOR3"
- note removed: "MOTOR4"
- note removed: "Micro Controller"
- note removed: "Motor Controller 1"
- note removed: "Motor Controller 2"
- note removed: "PWMA\nAIN2\nAIN1\nSTBY\nBIN1\nBIN2\nPWMB\nGND"
- note removed: "RST\nB11\nB10\nB1\nB0\nA7\nA6\nA5\nA4\nNC\nA3\nA2\nA1\nA0\nC13\nC14\nC15\nVBAT"
- note removed: "SWITCH"
- note removed: "VM\nVCC\nGND\nA01\nA02\nB02\nB01\nGND"
- moved on the sheet: J23, J9

Commit message: v2提交
Parts:
- C19, C20, C21, C22: footprint Capacitor_SMD:C_0603_1608Metric -> Capacitor_SMD:C_0402_1005Metric
- C23, C24, C25, C26, C27, C28: footprint Capacitor_SMD:C_0805_2012Metric -> Capacitor_SMD:C_0402_1005Metric
- D5: value LED_Red -> LED_White
- J9: footprint Connector_PinHeader_2.54mm:PinHeader_2x04_P2.54mm_Vertical -> Connector_PinHeader_2.54mm:PinHeader_1x04_P2.54mm_Vertical; symbol Connector_Generic:Conn_02x04_Odd_Even -> Connector_Generic:Conn_01x04
- R12, R13, R14, R15, R16, R17, R18, R19, R20: footprint Resistor_SMD:R_0805_2012Metric -> Resistor_SMD:R_0402_1005Metric
- Y1: footprint Crystal:Crystal_C38-LF_D3.0mm_L8.0mm_Horizontal -> Crystal:Crystal_SMD_3215-2Pin_3.2x1.5mm
- Y2: footprint Crystal:Crystal_SMD_5032-2Pin_5.0x3.2mm -> Crystal:Crystal_SMD_3225-4Pin_3.2x2.5mm; symbol Device:Crystal -> Device:Crystal_GND24
Connections:
- net labels removed: +5VA
- wire segments 40 -> 48
- no-connect marks 7 -> 6
Other:
- moved on the sheet: C26, D5, R17, R18, R20

Commit message: Modify some footprints.
Parts:
- J2: symbol Connector:USB_C_Receptacle_USB2.0 -> BaseBoard-rescue:USB_C_Receptacle_USB2.0-Connector
- Y2: footprint Crystal:Crystal_SMD_3225-4Pin_3.2x2.5mm -> Crystal:Crystal_SMD_5032-4Pin_5.0x3.2mm
Changed lines of the file:
@@
 $EndComp
 $Comp
-L Connector:USB_C_Receptacle_USB2.0 J2
+L BaseBoard-rescue:USB_C_Receptacle_USB2.0-Connector J2
 U 1 1 61491E1C
 P 4250 1600
@@
 F 0 "Y2" H 4400 3968 50  0000 C CNN
 F 1 "8Mhz" H 4400 3877 50  0000 C CNN
-F 2 "Crystal:Crystal_SMD_3225-4Pin_3.2x2.5mm" H 4400 3700 50  0001 C CNN
+F 2 "Crystal:Crystal_SMD_5032-4Pin_5.0x3.2mm" H 4400 3700 50  0001 C CNN
 F 3 "~" H 4400 3700 50  0001 C CNN
 	1    4400 3700
