File: BaseBoard/BaseBoard.kicad_pcb (KiCad board)
At the start: 2 copper layers, 100 x 86 mm, 105 parts, among them J1 Raspberry_Pi_2_3, J10 MOTOR, J14 Conn_01x02_Female, J15 Conn_01x02_Female, J16 Conn_01x02_Female, J2 USB_C_Receptacle_USB2.0, J21 Conn_01x02_Female, J22 USB_C_Receptacle_USB2.0, J23 IMU, J3 Conn_01x04, J4 MOTOR, J5 Barrel_Jack_Switch, J7 MOTOR, J8 MOTOR, J9 Conn_02x04, K1 SRD-12V, Q1 9926A, SW1 SW_Push, SW2 SW_Push, U1 CH224K, U2 CN3306, U3 XL4005, U4 TB6612FNG, U5 TB6612FNG, U6 GD32VF103Cx, U7 XC6206PxxxMR, Y1 32.768k, Y2 8Mhz

Commit message: V3 Baseboard
Parts:
- removed the C1 at (184.9, 84.8)
- removed the C16 at (132.0, 117.7)
- removed the C17 at (137.1, 121.5)
- removed C18: 100nF, Capacitor_SMD:C_0402_1005Metric
- removed C19, C21: 6pF, Capacitor_SMD:C_0402_1005Metric
- removed the C2 at (184.3, 76.3)
- removed C29: 10uF, Capacitor_SMD:C_0603_1608Metric
- removed the C3 at (171.7, 77.3)
- removed C30: 100pF, Capacitor_SMD:C_0402_1005Metric
- removed C31: 1uF, Capacitor_SMD:C_0402_1005Metric
- removed C32: 470uF, Capacitor_SMD:CP_Elec_10x10.5
- removed the C4 at (171.5, 75.3)
- removed the C5 at (152.1, 80.9)
- removed the C6 at (147.2, 74.7)
- removed the C7 at (160.9, 91.2)
- removed the C8 at (139.3, 95.2)
- removed the D1 at (175.6, 64.4)
- removed D2: LED_Green, LED_SMD:LED_0805_2012Metric
- removed D3, D4: SS54, Diode_SMD:D_SMA
- removed G***: LOGO, Customv2:Linux_12x12
- removed G***: LOGO, Customv2:ROS_LOGO_20x6
- removed G***: LOGO, Customv2:Anaheim_Electronic_20
- removed the J10 at (133.5, 145.6)
- removed J21: Conn_01x02_Female, Connector_Molex:Molex_Mini-Fit_Jr_5566-02A_2x01_P4.20mm_Vertical
- removed J22: USB_C_Receptacle_USB2.0, Connector_USB:USB_C_Receptacle_HRO_TYPE-C-31-M-12
- removed J23: IMU, Connector_PinSocket_2.54mm:PinSocket_1x08_P2.54mm_Vertical
- removed L1: 4.7uH, Inductor_SMD:L_7.3x7.3_H4.5
- removed L2: 33uH, Inductor_SMD:L_10.4x10.4_H4.8
- removed Q1: 9926A, Package_SO:SO-8_3.9x4.9mm_P1.27mm
- removed the R1 at (184.3, 74.2)
- removed R11: 360k, Resistor_SMD:R_0603_1608Metric
- removed R17, R18: 0, Resistor_SMD:R_0402_1005Metric
- removed R21: 1.6k, Resistor_SMD:R_0603_1608Metric
- removed R22: 95.3k, Resistor_SMD:R_0603_1608Metric
- removed R23: 910k, Resistor_SMD:R_0603_1608Metric
- removed R24: 1k, Resistor_SMD:R_0402_1005Metric
- removed R25: 0.02R, Resistor_SMD:R_2512_6332Metric
- removed R26: 0.05R/2W, Resistor_SMD:R_2512_6332Metric
- removed the R3 at (167.7, 75.8)
- removed the R4 at (177.9, 68.0)
- removed the R5 at (175.2, 75.2)
- removed the R6 at (175.2, 73.3)
- removed the R7 at (175.6, 68.0)
- removed the R8 at (157.1, 91.2)
- removed the U1 at (179.8, 73.8)
- removed the Y1 at (130.9, 94.9)
- added J1: IMU, Connector_PinSocket_2.54mm:PinSocket_1x10_P2.54mm_Vertical, F.Cu at (153.9, 101.0)
- added LOGO1: Logo_ROS, User_Symbol:ROS_LOGO_20x6, F.Cu at (203.0, 130.0)
- added LOGO2: Logo_Linux, User_Symbol:Linux_12x12, F.Cu at (205.0, 109.0)
- added LOGO3: Logo_Anaheim_Electronic, User_Symbol:Anaheim_Electronic_20, F.Cu at (172.1, 125.9)
- C1: renamed from C20; footprint Capacitor_SMD:C_0402_1005Metric -> Capacitor_SMD:C_0805_2012Metric
- C10: value 100nF -> 47uF; footprint Capacitor_SMD:C_0402_1005Metric -> Capacitor_SMD:CP_Elec_4x5.4
- C11: value 10uF -> 47uF
- C12, C14: footprint Capacitor_SMD:C_0402_1005Metric -> Capacitor_SMD:C_0805_2012Metric
- C13, C15: value 10uF -> 100nF; footprint Capacitor_SMD:CP_Elec_4x5.4 -> Capacitor_SMD:C_0805_2012Metric
- C16: renamed from C33; footprint Capacitor_SMD:C_0402_1005Metric -> Capacitor_SMD:C_0805_2012Metric
- C17: renamed from C34; footprint Capacitor_SMD:C_0402_1005Metric -> Capacitor_SMD:C_0805_2012Metric
- C2: renamed from C22; footprint Capacitor_SMD:C_0402_1005Metric -> Capacitor_SMD:C_0805_2012Metric
- C3: renamed from C23; footprint Capacitor_SMD:C_0402_1005Metric -> Capacitor_SMD:C_0805_2012Metric
- C4: renamed from C24; footprint Capacitor_SMD:C_0402_1005Metric -> Capacitor_SMD:C_0805_2012Metric
- C5: renamed from C25; footprint Capacitor_SMD:C_0402_1005Metric -> Capacitor_SMD:C_0805_2012Metric
- C6: renamed from C27; footprint Capacitor_SMD:C_0402_1005Metric -> Capacitor_SMD:C_0805_2012Metric
- C7: renamed from C26; footprint Capacitor_SMD:C_0402_1005Metric -> Capacitor_SMD:C_0805_2012Metric
- C8: renamed from C28; footprint Capacitor_SMD:C_0402_1005Metric -> Capacitor_SMD:C_0805_2012Metric
- C9: value 1uF -> 47uF; footprint Capacitor_SMD:C_0402_1005Metric -> Capacitor_SMD:CP_Elec_4x5.4
- J10: renamed from J14; footprint Connector_Molex:Molex_Mini-Fit_Jr_5566-02A_2x01_P4.20mm_Vertical -> Connector_JST:JST_EH_S2B-EH_1x02_P2.50mm_Horizontal; moved to B.Cu
- J11: renamed from J15; footprint Connector_Molex:Molex_Mini-Fit_Jr_5566-02A_2x01_P4.20mm_Vertical -> Connector_Molex:Molex_Mini-Fit_Jr_5569-02A2_2x01_P4.20mm_Horizontal; moved to B.Cu
- J12: renamed from J16; footprint Connector_AMASS:AMASS_XT60-M_1x02_P7.20mm_Vertical -> Connector_AMASS:AMASS_XT30PW-M_1x02_P2.50mm_Horizontal; moved to B.Cu
- J2: renamed from J3; footprint Connector_JST:JST_PH_B4B-PH-K_1x04_P2.00mm_Vertical -> Connector_JST:JST_XH_B4B-XH-A_1x04_P2.50mm_Vertical
- J5: renamed from J9; footprint Connector_PinHeader_2.54mm:PinHeader_1x04_P2.54mm_Vertical -> Connector_PinHeader_2.54mm:PinHeader_1x04_P2.54mm_Horizontal; moved to B.Cu
- J6: renamed from J4; footprint Connector_JST:JST_PH_B6B-PH-K_1x06_P2.00mm_Vertical -> Connector_JST:JST_PH_S6B-PH-K_1x06_P2.00mm_Horizontal
- J7, J8: footprint Connector_JST:JST_PH_B6B-PH-K_1x06_P2.00mm_Vertical -> Connector_JST:JST_PH_S6B-PH-K_1x06_P2.00mm_Horizontal
- J9: renamed from J5; moved to B.Cu
- K1: moved to B.Cu
- R1: renamed from R12; footprint Resistor_SMD:R_0402_1005Metric -> Resistor_SMD:R_0805_2012Metric
- R10: footprint Resistor_SMD:R_0402_1005Metric -> Resistor_SMD:R_0805_2012Metric
- R2: value 820k -> 5.1k; footprint Resistor_SMD:R_0603_1608Metric -> Resistor_SMD:R_0805_2012Metric
- R3: renamed from R13; footprint Resistor_SMD:R_0402_1005Metric -> Resistor_SMD:R_0805_2012Metric
- R4: renamed from R14; footprint Resistor_SMD:R_0402_1005Metric -> Resistor_SMD:R_0805_2012Metric
- R5: renamed from R15; footprint Resistor_SMD:R_0402_1005Metric -> Resistor_SMD:R_0805_2012Metric
- R6: renamed from R16; footprint Resistor_SMD:R_0402_1005Metric -> Resistor_SMD:R_0805_2012Metric
- R7: renamed from R19; footprint Resistor_SMD:R_0402_1005Metric -> Resistor_SMD:R_0805_2012Metric
- R8: renamed from R20; footprint Resistor_SMD:R_0402_1005Metric -> Resistor_SMD:R_0805_2012Metric
- R9: value 2k -> 360k; footprint Resistor_SMD:R_0603_1608Metric -> Resistor_SMD:R_0805_2012Metric
- SW1, SW2: footprint Button_Switch_SMD:SW_SPST_TL3342 -> User_Button_Switch:SW_SPST_EVQP7C-Single
- U2: value CN3306 -> DRV8870DDA; footprint Package_SO:TSSOP-16_4.4x5mm_P0.65mm -> Package_SO:Texas_HTSOP-8-1EP_3.9x4.9mm_P1.27mm_EP2.95x4.9mm_Mask2.4x3.1mm_ThermalVias
- U3: value XL4005 -> DRV8870DDA; footprint Package_TO_SOT_SMD:TO-263-5_TabPin3 -> Package_SO:Texas_HTSOP-8-1EP_3.9x4.9mm_P1.27mm_EP2.95x4.9mm_Mask2.4x3.1mm_ThermalVias
- U4: value TB6612FNG -> DRV8870DDA; footprint Package_SO:SSOP-24_5.3x8.2mm_P0.65mm -> Package_SO:Texas_HTSOP-8-1EP_3.9x4.9mm_P1.27mm_EP2.95x4.9mm_Mask2.4x3.1mm_ThermalVias
- U5: value TB6612FNG -> MINI560; footprint Package_SO:SSOP-24_5.3x8.2mm_P0.65mm -> User_Module:Converter_DCDC_Mini_560
- U6: renamed from U7; value XC6206PxxxMR -> AMS1117-3.3; footprint Package_TO_SOT_SMD:SOT-23 -> Package_TO_SOT_SMD:SOT-223-3_TabPin2
- Y1: renamed from Y2; footprint Crystal:Crystal_SMD_5032-4Pin_5.0x3.2mm -> Crystal:Crystal_SMD_3225-4Pin_3.2x2.5mm
- moved J9 95.5 mm to (124.5, 135.0), turned to 180 degrees
- moved J12 91.5 mm to (124.2, 126.0), turned to -90 degrees
- moved J6 91.2 mm to (198.5, 70.8), turned to 180 degrees
- moved J4 87.8 mm to (208.2, 87.5), turned to 90 degrees
- moved J7 84.4 mm to (182.5, 70.8), turned to 180 degrees
- moved C12 84.1 mm to (199.6, 81.2), turned to -90 degrees
- moved R1 84.0 mm to (200.6, 90.4)
- moved J8 83.3 mm to (166.5, 70.8), turned to 180 degrees
- moved R7 82.0 mm to (202.9, 76.4), turned to 90 degrees
- moved C8 81.0 mm to (202.9, 79.8), turned to -90 degrees
- moved R3 80.4 mm to (200.6, 88.4)
- moved C13 77.3 mm to (192.0, 81.2), turned to -90 degrees
- moved R4 77.1 mm to (200.6, 86.4), turned to 0 degrees
- moved C10 64.3 mm to (198.2, 76.0), turned to 90 degrees
- moved SW2 62.9 mm to (208.8, 78.8), turned to 90 degrees
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- renumbered D5 to D1, J1 to J3, J2 to J4, U6 to U1
Connections:
- C10 pad 1: /ADC -> +12VA
- C11 pad 1: +3V3 -> +12VA
- C12 pad 1: +3V3 -> +12VA
- C15 pad 1: +3V3 -> /ADC
- C7 pad 1: /VSSA -> GND
- C7 pad 2: /VDDA -> +3V3
- C9 pad 1: +5V -> +12VA
- J3 pad 11: Net-(J1-Pad11) -> unconnected-(J3-Pad11)
- J3 pad 12: Net-(J1-Pad12) -> unconnected-(J3-Pad12)
- J3 pad 13: Net-(J1-Pad13) -> unconnected-(J3-Pad13)
- J3 pad 19: Net-(J1-Pad19) -> /GPIO10
- J3 pad 23: Net-(J1-Pad23) -> /GPIO11
- J3 pad 26: Net-(J1-Pad26) -> unconnected-(J3-Pad26)
- J3 pad 27: Net-(J1-Pad27) -> unconnected-(J3-Pad27)
- J3 pad 28: Net-(J1-Pad28) -> unconnected-(J3-Pad28)
- J3 pad 29: Net-(J1-Pad29) -> unconnected-(J3-Pad29)
- J3 pad 31: Net-(J1-Pad31) -> unconnected-(J3-Pad31)
- J3 pad 32: Net-(J1-Pad32) -> unconnected-(J3-Pad32)
- J3 pad 33: Net-(J1-Pad33) -> unconnected-(J3-Pad33)
- J3 pad 35: Net-(J1-Pad35) -> unconnected-(J3-Pad35)
- J3 pad 36: Net-(J1-Pad36) -> unconnected-(J3-Pad36)
- J3 pad 37: Net-(J1-Pad37) -> unconnected-(J3-Pad37)
- J3 pad 38: Net-(J1-Pad38) -> unconnected-(J3-Pad38)
- J3 pad 40: Net-(J1-Pad40) -> unconnected-(J3-Pad40)
- J3 pad 7: Net-(J1-Pad7) -> unconnected-(J3-Pad7)
- J4 pad A5: Net-(J2-PadA5) -> Net-(J4-PadA5)
- J4 pad A8: Net-(J2-PadA8) -> unconnected-(J4-PadA8)
- J4 pad B5: Net-(J2-PadA5) -> Net-(J4-PadB5)
- J4 pad B8: Net-(J2-PadB8) -> unconnected-(J4-PadB8)
- J5 pad 1: GND -> +3V3
- J5 pad 2: /DEBUG_RX -> /DEBUG_TX
- J5 pad 3: /DEBUG_TX -> /DEBUG_RX
- J5 pad 4: +3V3 -> GND
- K1 pad 4: Net-(K1-Pad4) -> unconnected-(K1-Pad4)
- R1 pad 2: Net-(J2-PadA5) -> Net-(J4-PadA5)
- R2 pad 1: VBUS -> GND
- R2 pad 2: Net-(R2-Pad2) -> Net-(J4-PadB5)
- R3 pad 1: /PWM4 -> /USB_DM
- R9 pad 1: Net-(C7-Pad2) -> +12V
- R9 pad 2: GND -> /ADC
- U1 pad 1: Net-(U6-Pad1) -> unconnected-(U1-Pad1)
- U1 pad 14: /MOT1_C1 -> unconnected-(U1-Pad14)
- U1 pad 15: /MOT1_C2 -> unconnected-(U1-Pad15)
- U1 pad 16: /MOT2_C1 -> unconnected-(U1-Pad16)
- U1 pad 17: /MOT2_C2 -> unconnected-(U1-Pad17)
- U1 pad 19: Net-(U6-Pad19) -> unconnected-(U1-Pad19)
- U1 pad 25: /MOT3_C1 -> unconnected-(U1-Pad25)
- U1 pad 26: /MOT3_C2 -> /PWM1_ON
- U1 pad 27: /MOT4_C1 -> /PWM2_ON
- U1 pad 28: /MOT4_C2 -> /PWM3_ON
- U1 pad 32: /PWM4 -> /USB_DM
- U1 pad 38: /ENC4_A -> /JTDI
- U1 pad 39: /ENC4_B -> /JTDO
- U1 pad 45: Net-(U6-Pad45) -> unconnected-(U1-Pad45)
- U1 pad 46: Net-(U6-Pad46) -> unconnected-(U1-Pad46)
- U1 pad 8: /VSSA -> GND
- U1 pad 9: /VDDA -> +3V3
- U2 pad 1: Net-(R22-Pad1) -> GND
- U2 pad 2: Net-(C3-Pad1) -> /PWM1_ON
- U2 pad 3: Net-(R2-Pad2) -> /PWM1
- U2 pad 4: Net-(U2-Pad4) -> +3V3
- U2 pad 5: GND -> +12VA
- U2 pad 6: Net-(D1-Pad1) (its old number) -> /Motor/MOT1_N
- U2 pad 7: Net-(D2-Pad1) -> GND
- U2 pad 8: Net-(C32-Pad1) -> /Motor/MOT1_P
- U2 pad 9: +BATT -> GND
- U3 pad 2: Net-(C7-Pad2) -> /PWM2_ON
- U3 pad 3: Net-(D4-Pad1) -> /PWM2
- U3 pad 4: +12V -> +3V3
- U3 pad 5: +12V -> +12VA
- U4 pad 1: /Motor/MOT1_N -> GND
- U4 pad 2: /Motor/MOT1_N -> /PWM3_ON
- U4 pad 3: GND -> /PWM3
- U4 pad 4: GND -> +3V3
- U4 pad 5: /Motor/MOT1_P -> +12VA
- U4 pad 6: /Motor/MOT1_P -> /Motor/MOT3_N
- U4 pad 7: /Motor/MOT2_P -> GND
- U4 pad 8: /Motor/MOT2_P -> /Motor/MOT3_P
- U5 pad 1: /Motor/MOT3_N -> +12V
- U5 pad 2: /Motor/MOT3_N -> GND
- U5 pad 3: GND -> +5V
Routing:
- net GND: track 188.9 -> 80.8 mm, vias 35 -> 11
- net VBUS: track 80.6 -> 0.00 mm
- net /PWM4: track 76.4 -> 0.00 mm, vias 6 -> 0
- net +BATT: track 112.6 -> 37.9 mm, vias 2 -> 0
- net Net-(D1-Pad1): track 92.5 -> 39.5 mm
- net /ENC4_A: track 47.6 -> 0.00 mm, vias 1 -> 0
- net /ENC4_B: track 47.1 -> 0.00 mm, vias 1 -> 0
- net +3V3: track 254.8 -> 209.8 mm, vias 15 -> 6
- net /BOOT0: track 80.8 -> 37.6 mm, vias 4 -> 2
- net Net-(C32-Pad1): track 40.7 -> 0.00 mm, vias 2 -> 0
- net /CTL_TX: track 50.6 -> 16.1 mm, vias 2 -> 0
- net /CTL_RX: track 49.6 -> 19.5 mm, vias 2 -> 0
- net /MOT3_C1: track 30.1 -> 0.00 mm, vias 2 -> 0
- net /MOT4_C1: track 29.7 -> 0.00 mm, vias 2 -> 0
- net Net-(D4-Pad1): track 29.2 -> 0.00 mm
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Other:
- net class Default removed
- net class Power removed
- net class Power2 removed
- board text added: "3V3 GND SCL SDA IO22 IO23 IO24 IO25 IO10 IO11"
- board text added: "Debug UART"
- board text added: "Motor"
- board text added: "Power"
- board text added: "Rpi Hat v3 ©2021-2022 ESAC"
- board text added: "Status"
- board text removed: "+"
- board text removed: "3V3 GND SCL SDA IO22 IO23 IO24 IO25"
- board text removed: "Motor 4"
- board text removed: "Stop"
- board text removed: "Switch"
- board text removed: "Work Charge Full"
- board text removed: "©2021 ESAC Rpi Motor Hat v2"
