File: BaseBoard/BaseBoard.kicad_pcb (KiCad board)
At the start: 2 copper layers, 100 x 86 mm, 60 parts, among them J1 IMU, J10 Conn_01x02_Female, J11 Conn_01x02_Female, J12 Conn_01x02_Female, J2 Conn_01x04, J3 Raspberry_Pi_2_3, J4 USB_C_Receptacle_USB2.0, J5 Conn_02x04, J6 MOTOR, J7 MOTOR, J8 MOTOR, J9 Barrel_Jack_Switch, K1 SRD-12V, SW1 SW_Push, SW2 SW_Push, U1 GD32VF103Cx, U2 DRV8870DDA, U3 DRV8870DDA, U4 DRV8870DDA, U5 MINI560, U6 AMS1117-3.3, Y1 8Mhz

Commit message: 使用功率地
Parts:
- added JP1: SolderJumper_2_Bridged, Jumper:SolderJumper-2_P1.3mm_Bridged2Bar_Pad1.0x1.5mm, F.Cu at (152.8, 84.0)
- U1: value GD32VF103Cx -> GD32VF103C8Tx
- moved C12 2.69 mm to (198.6, 78.7), turned to 0 degrees
- moved C11 2.69 mm to (160.4, 76.5)
- moved C13 2.67 mm to (191.1, 78.7), turned to 0 degrees
- moved U4 1.84 mm to (157.2, 84.0)
- moved C17 1.35 mm to (151.1, 72.6)
- moved C16 1.30 mm to (151.1, 78.0)
- moved U6 1.30 mm to (146.5, 75.3)
- moved C14 1.26 mm to (161.7, 80.8), turned to 0 degrees
- moved C8 1.17 mm to (203.9, 80.4)
- moved D1 1.17 mm to (203.9, 70.2)
- moved R7 1.17 mm to (203.9, 77.0)
- moved R8 1.17 mm to (203.9, 73.6)
- moved C9 1.04 mm to (189.6, 75.3), turned to 0 degrees
- moved C10 0.99 mm to (198.9, 75.3), turned to 0 degrees
- moved U2 0.40 mm to (195.8, 84.0)
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Connections:
- C10 pad 2: GND -> GNDPWR
- C11 pad 2: GND -> GNDPWR
- C12 pad 2: GND -> GNDPWR
- C13 pad 2: GND -> GNDPWR
- C14 pad 2: GND -> GNDPWR
- C9 pad 2: GND -> GNDPWR
- SW1 pad 1: /BOOT0 -> +3V3
- SW1 pad 2: +3V3 -> /BOOT0
- U1 pad 1: unconnected-(U1-Pad1) -> +3V3
- U2 pad 1: GND -> GNDPWR
- U2 pad 7: GND -> GNDPWR
- U2 pad 9: GND -> GNDPWR
- U3 pad 1: GND -> GNDPWR
- U3 pad 7: GND -> GNDPWR
- U3 pad 9: GND -> GNDPWR
- U4 pad 1: GND -> GNDPWR
- U4 pad 7: GND -> GNDPWR
- U4 pad 9: GND -> GNDPWR
Routing:
- net +12VA: track 134.4 -> 62.3 mm
- net GND: track 80.8 -> 110.6 mm, vias 11 -> 16
- net GNDPWR: track 0.00 -> 19.7 mm
- net /ENC3_A: track 39.2 -> 29.9 mm
- net /ENC3_B: track 37.1 -> 28.1 mm
- net Net-(C8-Pad1): track 39.3 -> 45.9 mm
- net /ENC2_A: track 11.8 -> 14.6 mm, vias 1 -> 0
- net /Motor/MOT3_N: track 15.8 -> 18.5 mm
- net /PWM3: track 26.3 -> 28.8 mm
- net +BATT: track 37.9 -> 35.8 mm
- net /PWM3_ON: track 27.8 -> 29.9 mm
- net /Motor/MOT3_P: track 15.0 -> 16.8 mm
- net /PWM1_ON: track 22.5 -> 24.0 mm
- net +5V: track 108.8 -> 107.7 mm, vias 1 -> 3
- net /PWM1: track 23.6 -> 24.8 mm
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- added copper zone on F.Cu, net +12VA
- added copper zone on B.Cu, net GNDPWR
- added copper zone on F.Cu, net GNDPWR
Other:
- board text added: "Rpi Hat v3 ©2021-2023 ESAC"
- board text added: "Stop"
- board text removed: "Motor"
- board text removed: "Rpi Hat v3 ©2021-2022 ESAC"

Commit message: 临时提交
Parts:
- added J13: Conn_01x02_Female, Connector_JST:JST_PH_S2B-PH-K_1x02_P2.00mm_Horizontal, B.Cu at (182.2, 69.5)
- added J14: Conn_01x03_Female, Connector_JST:JST_PH_S3B-PH-K_1x03_P2.00mm_Horizontal, B.Cu at (122.4, 69.4)
- added R11: 10k, Resistor_SMD:R_0805_2012Metric, B.Cu at (161.4, 88.3)
- C1, C10, C11, C12, C13, C14, C15, C16, C17, C2, C3, C4, C5, C6, C7, C8, C9, D1, J4, J6, J7, J8, R1, R10, R2, R3, R4, R5, R6, R7, R8, R9, SW1, SW2, U1, U2, U3, U4, U5, U6, Y1: moved to B.Cu
- J10: footprint Connector_JST:JST_EH_S2B-EH_1x02_P2.50mm_Horizontal -> Connector_JST:JST_PH_S2B-PH-K_1x02_P2.00mm_Horizontal
- J11: footprint Connector_Molex:Molex_Mini-Fit_Jr_5569-02A2_2x01_P4.20mm_Horizontal -> Connector_Molex:Molex_KK-396_A-41792-0002_1x02_P3.96mm_Horizontal
- J2: footprint Connector_JST:JST_XH_B4B-XH-A_1x04_P2.50mm_Vertical -> Connector_JST:JST_PH_S4B-PH-K_1x04_P2.00mm_Horizontal; moved to B.Cu
- moved C10 70.6 mm to (128.3, 73.8), turned to 180 degrees
- moved C12 69.5 mm to (129.1, 77.2), turned to 180 degrees
- moved J6 66.6 mm to (131.9, 69.4), turned to 0 degrees
- moved U2 63.8 mm to (132.0, 82.5)
- moved C13 51.2 mm to (139.9, 77.2), turned to 180 degrees
- moved C9 50.6 mm to (139.0, 73.8), turned to 180 degrees
- moved U3 45.4 mm to (142.8, 82.5)
- moved C15 36.3 mm to (124.5, 114.9)
- moved J7 35.3 mm to (147.2, 69.4), turned to 0 degrees
- moved J2 33.8 mm to (189.9, 69.4), turned to 0 degrees
- moved R10 33.1 mm to (124.5, 112.9)
- moved R9 30.2 mm to (124.5, 110.9)
- moved J10 29.5 mm to (117.3, 113.9), turned to 90 degrees
- moved R8 28.6 mm to (176.0, 67.2)
- moved C17 27.7 mm to (130.7, 91.4)
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Connections:
- net /USB_DM renamed /PWM4
- C8 pad 1: Net-(C8-Pad1) -> Net-(U1-NRST)
- R7 pad 1: Net-(C8-Pad1) -> Net-(U1-NRST)
- SW1 pad 1: +3V3 -> /BOOT0
- SW1 pad 2: /BOOT0 -> +3V3
- SW2 pad 1: GND -> Net-(U1-NRST)
- SW2 pad 2: Net-(C8-Pad1) -> GND
- U1 pad 25: unconnected-(U1-Pad25) -> /BREAK
- U1 pad 7: Net-(C8-Pad1) -> Net-(U1-NRST)
Routing:
- net +5V: track 107.7 -> 197.2 mm
- net /PWM4: track 25.0 -> 84.9 mm, vias 0 -> 3
- net GND: track 110.6 -> 55.3 mm, vias 16 -> 3
- net Net-(C8-Pad1): track 45.9 -> 0.00 mm, vias 2 -> 0
- net Net-(U1-NRST): track 0.00 -> 44.5 mm, vias 0 -> 2
- net +12VA: track 62.3 -> 18.2 mm
- net +12V: track 83.6 -> 48.8 mm, vias 1 -> 0
- net /BREAK: track 0.00 -> 34.2 mm, vias 0 -> 1
- net /ADC: track 41.6 -> 9.31 mm, vias 2 -> 1
- net +3V3: track 209.4 -> 236.6 mm, vias 7 -> 9
- net /LIDAR_TX: track 8.05 -> 35.1 mm, vias 0 -> 2
- net Net-(D1-K): track 38.9 -> 15.0 mm, vias 2 -> 0
- net /LIDAR_RX: track 10.6 -> 29.6 mm, vias 0 -> 2
- net /ENC1_B: track 20.5 -> 37.0 mm
- net /PWM2_ON: track 14.0 -> 29.9 mm
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- added copper zone on B.Cu, net +12VA
- removed copper zone on F.Cu, net +12VA

Commit message: 更新V3线路板
Parts:
- added C18: 100nF, Capacitor_SMD:C_0805_2012Metric, B.Cu at (119.6, 145.6)
- added C19: 100nF, Capacitor_SMD:C_0805_2012Metric, B.Cu at (122.0, 134.5)
- added C20: 100nF, Capacitor_SMD:C_0805_2012Metric, B.Cu at (120.7, 131.5)
- added C21: 100nF, Capacitor_SMD:C_0805_2012Metric, B.Cu at (123.3, 131.5)
- added C22: 100nF, Capacitor_SMD:C_0805_2012Metric, B.Cu at (121.7, 145.6)
- added C23: 3.3nF, Capacitor_SMD:C_0805_2012Metric, B.Cu at (123.8, 145.6)
- added J15: HT396R_1x02, Connector_Molex:Molex_KK-396_A-41792-0002_1x02_P3.96mm_Horizontal, B.Cu at (139.5, 139.5)
- added JP2: NC, Jumper:SolderJumper-2_P1.3mm_Bridged2Bar_Pad1.0x1.5mm, B.Cu at (114.1, 125.9)
- added Q1: 2N7002, Package_TO_SOT_SMD:SOT-23, B.Cu at (114.0, 136.9)
- added R12: 10mR, Resistor_SMD:R_1210_3225Metric, B.Cu at (122.0, 124.2)
- added R13: 100, Resistor_SMD:R_0805_2012Metric, B.Cu at (120.7, 127.9)
- added R14: 100, Resistor_SMD:R_0805_2012Metric, B.Cu at (123.3, 127.9)
- added R15: 220k, Resistor_SMD:R_0805_2012Metric, B.Cu at (116.8, 136.8)
- added R16: 100k, Resistor_SMD:R_0805_2012Metric, B.Cu at (116.8, 140.2)
- added R17: 220k, Resistor_SMD:R_0805_2012Metric, B.Cu at (118.8, 136.8)
- added R18: 16.5k, Resistor_SMD:R_0805_2012Metric, B.Cu at (118.8, 140.2)
- added U7: BMI088, Smallbot:Bochs_LGA16_2x7+2x1, B.Cu at (177.4, 102.4)
- added U8: BQ34Z100, Package_SO:TSSOP-14_4.4x5mm_P0.65mm, B.Cu at (122.6, 139.4)
- J1: value IMU -> PH2.0_1x03; footprint Connector_PinSocket_2.54mm:PinSocket_1x10_P2.54mm_Vertical -> Connector_JST:JST_PH_S3B-PH-K_1x03_P2.00mm_Horizontal; moved to B.Cu
- J11: value Conn_01x02_Female -> HT396R_1x02
- J12: value Conn_01x02_Female -> XT30PW
- J14: value Conn_01x03_Female -> PH2.0_1x03
- J2: value Conn_01x04 -> PH2.0_1x04
- J5: value Conn_02x04 -> PinHeader_2.54_1x04
- J6, J7, J8: value MOTOR -> PH2.0_1x06
- JP1: value SolderJumper_2_Bridged -> NC; moved to B.Cu
- SW1, SW2: value SW_Push -> TL3342; footprint User_Button_Switch:SW_SPST_EVQP7C-Single -> Button_Switch_SMD:SW_SPST_TL3342
- moved J1 48.2 mm to (117.5, 132.6)
- moved J10 44.4 mm to (120.0, 69.6), turned to 0 degrees
- moved R9 33.8 mm to (131.7, 77.8)
- moved C15 33.5 mm to (131.7, 82.1)
- moved R10 33.5 mm to (131.7, 80.1)
- moved R8 24.6 mm to (200.6, 67.1), turned to 0 degrees
- moved D1 22.5 mm to (200.6, 65.1), turned to 0 degrees
- moved C7 17.5 mm to (192.7, 84.7)
- moved C3 17.4 mm to (179.0, 79.0)
- moved C4 17.4 mm to (194.7, 84.7)
- moved C1 17.4 mm to (193.8, 75.4)
- moved C2 17.4 mm to (193.8, 81.7)
- moved C5 17.4 mm to (189.1, 75.7)
- moved C6 17.4 mm to (182.0, 88.9)
- moved R11 17.4 mm to (178.8, 88.2)
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Connections:
- J1 pad 1: +3.3VA -> /I2C_SCL
- J1 pad 2: GND -> /I2C_SDA
- J1 pad 3: /SCL -> GNDA
- J12 pad 1: GND -> -BATT
- J14 pad 1: +12VA -> GND
- J14 pad 3: GNDPWR -> +12VA
- J3 pad 15: /GPIO22 -> unconnected-(J3-GPIO22-Pad15)
- J3 pad 16: /GPIO23 -> unconnected-(J3-GPIO23-Pad16)
- J3 pad 18: /GPIO24 -> /IMU_INT2
- J3 pad 19: /GPIO10 -> /SPI_MOSI
- J3 pad 21: /LIDAR_TX -> /SPI_MISO
- J3 pad 22: /GPIO25 -> /IMU_INT1
- J3 pad 23: /GPIO11 -> /SPI_CLK
- J3 pad 24: /LIDAR_RX -> /SPI_CS1
- J3 pad 26: unconnected-(J3-~{CE1}/GPIO7-Pad26) -> /SPI_CS2
- J3 pad 29: unconnected-(J3-GCLK1/GPIO5-Pad29) -> /LIDAR_TX
- J3 pad 3: /SDA -> unconnected-(J3-SDA/GPIO2-Pad3)
- J3 pad 5: /SCL -> unconnected-(J3-SCL/GPIO3-Pad5)
- J3 pad 7: unconnected-(J3-GCLK0/GPIO4-Pad7) -> /LIDAR_RX
- U1 pad 45: unconnected-(U1-PB8-Pad45) -> /I2C_SCL
- U1 pad 46: unconnected-(U1-PB9-Pad46) -> /I2C_SDA
Routing:
- net /I2C_SDA: track 0.00 -> 152.1 mm, vias 0 -> 4
- net /I2C_SCL: track 0.00 -> 149.7 mm, vias 0 -> 4
- net /ADC: track 9.31 -> 75.7 mm, vias 1 -> 2
- net GND: track 55.3 -> 98.9 mm, vias 3 -> 16
- net /LIDAR_RX: track 29.6 -> 57.2 mm, vias 2 -> 1
- net /DEBUG_RX: track 56.1 -> 78.3 mm, vias 0 -> 1
- net Net-(U1-NRST): track 44.5 -> 23.5 mm, vias 2 -> 0
- net /SPI_CS2: track 0.00 -> 20.9 mm
- net /DEBUG_TX: track 63.0 -> 83.7 mm, vias 1 -> 2
- net +3V3: track 236.6 -> 255.7 mm, vias 9 -> 8
- net /CTL_RX: track 14.8 -> 32.3 mm, vias 1 -> 0
- net /CTL_TX: track 16.2 -> 33.2 mm, vias 1 -> 0
- net /USB_DP: track 37.7 -> 20.8 mm
- net Net-(Q1-S): track 0.00 -> 16.9 mm
- net +3.3VA: track 3.61 -> 20.0 mm, vias 0 -> 2
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- added copper zone on F.Cu, net +12V
- added copper zone on F.Cu, net +BATT
- added copper zone on B.Cu, net -BATT
- added copper zone on B.Cu, net GNDA
- added copper zone on F.Cu, net GNDA
Other:
- board text added: "+ 12.6V -"
- board text added: "+ PWM -"
- board text added: "12V CTL"
- board text added: "Boot"
- board text added: "Break"
- board text added: "Button"
- board text added: "DC-2.1/5.5"
- board text added: "DFU"
- board text added: "GND A 3V3 B + -"
- board text added: "GND SDA SCL"
- board text added: "GND SIG"
- board text added: "Gauge"
- board text added: "Internal"
- board text added: "J14"
- board text added: "LED"
- board text added: "LiDAR"
- board text added: "Motor 4"
- board text added: "Switch"
- board text added: "USB-C"
- board text removed: "3V3 GND SCL SDA IO22 IO23 IO24 IO25 IO10 IO11"
- board text removed: "Boot0"
- board text removed: "GND ENCA 3V3 ENCB MOT+ MOT-"
- board text removed: "IMU"
- board text removed: "Lidar"

Commit message: 添加v3初版设计
Parts:
- removed U6: AMS1117-3.3, Package_TO_SOT_SMD:SOT-223-3_TabPin2
- added C16: 100nF, Capacitor_SMD:C_0805_2012Metric, B.Cu at (136.9, 97.0)
- added REF**: Symbol_Barrel_Polarity, Symbol:Symbol_Barrel_Polarity, F.Cu at (122.4, 146.0)
- added U7: SGM2028-3.3YN5G, Package_TO_SOT_SMD:SOT-23-5, B.Cu at (140.0, 95.2)
- ? (x4): footprint RPi_Hat:RPi_Hat_Mounting_Hole -> BaseBoard:RPi_Hat_Mounting_Hole
- LOGO1: footprint User_Symbol:ROS_LOGO_20x6 -> BaseBoard:ROS_LOGO_20x6
- LOGO2: footprint User_Symbol:Linux_12x12 -> BaseBoard:Linux_12x12
- LOGO3: footprint User_Symbol:Anaheim_Electronic_20 -> BaseBoard:Anaheim_Electronic_20
- REF** (x3): footprint MountingHole:MountingHole_3.2mm_M3_DIN965_Pad -> BaseBoard:MountingHole_3.2mm_M3_DIN965_Pad
- U5: footprint User_Module:Converter_DCDC_Mini_560 -> BaseBoard:Converter_DCDC_Mini_560
- moved C17 6.56 mm to (136.9, 93.5)
- moved C15 1.08 mm to (143.1, 95.2)
- renumbered C16 to C15, C15 to C18, C22 to C19, C19 to C21, C21 to C22, C18 to C23, C23 to C24, J2 to J1, J9 to J10, J10 to J11, J11 to J12, J12 to J13, J15 to J14, J1 to J15, J3 to J2, J4 to J3, J5 to J4, J13 to J5, J14 to J6, J6 to J7, J7 to J8, J8 to J9, R9 to R10, R10 to R11, R15 to R12, R16 to R13, R13 to R14, R12 to R15, R14 to R16, R8 to R7, R7 to R8, R11 to R9, U7 to U1, U1 to U2, U2 to U3, U3 to U4, U4 to U5
Routing:
- net GND: track 98.9 -> 93.4 mm, vias 16 -> 15
- net +3V3: track 255.7 -> 253.2 mm
- net Net-(U7-BP): track 0.00 -> 2.02 mm
- net +5V: track 187.7 -> 189.3 mm
- net /Motor/MOT1_P: track 13.6 -> 14.2 mm
Other:
- board text added: "+"
- board text added: "-"
- board text added: "DC 5.5-2.1"
- board text added: "DC Definition"
- board text removed: "DC-2.1/5.5"
