File: BaseBoard/Motor.kicad_sch (KiCad schematic)
At the start: 12 parts, among them J6 MOTOR, J7 MOTOR, J8 MOTOR, U2 DRV8870DDA, U3 DRV8870DDA, U4 DRV8870DDA

Commit message: 使用功率地
Connections:
- net GND: no longer C10.2, C11.2, C12.2, C13.2, C14.2, C9.2, U2.1 (GND), U2.7 (ISEN), U2.9 (GND), U3.1 (GND), U3.7 (ISEN), U3.9 (GND), U4.1 (GND), U4.7 (ISEN), U4.9 (GND)
- new net GNDPWR: C10.2, C11.2, C12.2, C13.2, C14.2, C9.2, U2.1 (GND), U2.7 (ISEN), U2.9 (GND), U3.1 (GND), U3.7 (ISEN), U3.9 (GND), U4.1 (GND), U4.7 (ISEN), U4.9 (GND)
Changed lines of the file:
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@@
-    (pin "1")
-  )
-  (symbol (lib_id "power:GND") (at 135.89 102.87 0) (unit 1)
-    (in_bom yes) (on_board yes)
-    (property "Reference" "#PWR061" (id 0) (at 135.89 109.22 0)
-      (effects (font (size 1.27 1.27)) hide)
-    )
-    (property "Value" "GND" (id 1) (at 136.017 107.2642 0))
-    (property "Footprint" "" (id 2) (at 135.89 102.87 0)
-      (effects (font (size 1.27 1.27)) hide)
-    )
-    (property "Datasheet" "" (id 3) (at 135.89 102.87 0)
-      (effects (font (size 1.27 1.27)) hide)
-    )
     (pin "1")
   )
@@
     (pin "9")
   )
-  (symbol (lib_id "power:GND") (at 123.19 66.04 0) (unit 1)
-    (in_bom yes) (on_board yes)
-    (property "Reference" "#PWR055" (id 0) (at 123.19 72.39 0)
-      (effects (font (size 1.27 1.27)) hide)
-    )
-    (property "Value" "GND" (id 1) (at 123.317 70.4342 0))
-    (property "Footprint" "" (id 2) (at 123.19 66.04 0)
-      (effects (font (size 1.27 1.27)) hide)
-    )
-    (property "Datasheet" "" (id 3) (at 123.19 66.04 0)
+  (symbol (lib_id "power:GNDPWR") (at 123.19 66.04 0) (unit 1)
+    (in_bom yes) (on_board yes) (fields_autoplaced)
+    (property "Reference" "#PWR0111" (id 0) (at 123.19 71.12 0)
+      (effects (font (size 1.27 1.27)) hide)
+    )
+    (property "Value" "GNDPWR" (id 1) (at 123.063 71.12 0))
+    (property "Footprint" "" (id 2) (at 123.19 67.31 0)
+      (effects (font (size 1.27 1.27)) hide)
+    )
+    (property "Datasheet" "" (id 3) (at 123.19 67.31 0)
+      (effects (font (size 1.27 1.27)) hide)
+    )
+    (pin "1")
+  )
+  (symbol (lib_id "power:GNDPWR") (at 135.89 102.87 0) (unit 1)
+    (in_bom yes) (on_board yes) (fields_autoplaced)
+    (property "Reference" "#PWR0109" (id 0) (at 135.89 107.95 0)
+      (effects (font (size 1.27 1.27)) hide)
+    )
+    (property "Value" "GNDPWR" (id 1) (at 135.763 107.95 0))
+    (property "Footprint" "" (id 2) (at 135.89 104.14 0)
+      (effects (font (size 1.27 1.27)) hide)
+    )
+    (property "Datasheet" "" (id 3) (at 135.89 104.14 0)
       (effects (font (size 1.27 1.27)) hide)
     )
@@
     (pin "1")
     (pin "2")
-  )
-  (symbol (lib_id "power:GND") (at 135.89 139.7 0) (unit 1)
-    (in_bom yes) (on_board yes)
-    (property "Reference" "#PWR062" (id 0) (at 135.89 146.05 0)
-      (effects (font (size 1.27 1.27)) hide)
-    )
-    (property "Value" "GND" (id 1) (at 136.017 144.0942 0))
-    (property "Footprint" "" (id 2) (at 135.89 139.7 0)
-      (effects (font (size 1.27 1.27)) hide)
-    )
-    (property "Datasheet" "" (id 3) (at 135.89 139.7 0)
-      (effects (font (size 1.27 1.27)) hide)
-    )
-    (pin "1")
   )
   (symbol (lib_id "power:+12VA") (at 123.19 45.72 0) (unit 1)
@@
     (pin "1")
   )
-  (symbol (lib_id "power:GND") (at 123.19 102.87 0) (unit 1)
-    (in_bom yes) (on_board yes)
-    (property "Reference" "#PWR057" (id 0) (at 123.19 109.22 0)
-      (effects (font (size 1.27 1.27)) hide)
-    )
-    (property "Value" "GND" (id 1) (at 123.317 107.2642 0))
-    (property "Footprint" "" (id 2) (at 123.19 102.87 0)
-      (effects (font (size 1.27 1.27)) hide)
-    )
-    (property "Datasheet" "" (id 3) (at 123.19 102.87 0)
-      (effects (font (size 1.27 1.27)) hide)
-    )
-    (pin "1")
-  )
   (symbol (lib_id "power:+3V3") (at 113.03 97.79 90) (unit 1)
     (in_bom yes) (on_board yes) (fields_autoplaced)
@@
     (pin "1")
     (pin "2")
-  )
-  (symbol (lib_id "power:GND") (at 123.19 139.7 0) (unit 1)
-    (in_bom yes) (on_board yes)
-    (property "Reference" "#PWR059" (id 0) (at 123.19 146.05 0)
-      (effects (font (size 1.27 1.27)) hide)
-    )
-    (property "Value" "GND" (id 1) (at 123.317 144.0942 0))
-    (property "Footprint" "" (id 2) (at 123.19 139.7 0)
-      (effects (font (size 1.27 1.27)) hide)
-    )
-    (property "Datasheet" "" (id 3) (at 123.19 139.7 0)
-      (effects (font (size 1.27 1.27)) hide)
-    )
-    (pin "1")
-  )
-  (symbol (lib_id "power:GND") (at 135.89 66.04 0) (unit 1)
-    (in_bom yes) (on_board yes)
-    (property "Reference" "#PWR060" (id 0) (at 135.89 72.39 0)
-      (effects (font (size 1.27 1.27)) hide)
-    )
-    (property "Value" "GND" (id 1) (at 136.017 70.4342 0))
-    (property "Footprint" "" (id 2) (at 135.89 66.04 0)
-      (effects (font (size 1.27 1.27)) hide)
-    )
-    (property "Datasheet" "" (id 3) (at 135.89 66.04 0)
-      (effects (font (size 1.27 1.27)) hide)
-    )
-    (pin "1")
   )
   (symbol (lib_id "power:+12VA") (at 123.19 119.38 0) (unit 1)
@@
     )
     (property "Datasheet" "" (id 3) (at 123.19 119.38 0)
+      (effects (font (size 1.27 1.27)) hide)
+    )
+    (pin "1")
+  )
+  (symbol (lib_id "power:GNDPWR") (at 123.19 102.87 0) (unit 1)
+    (in_bom yes) (on_board yes) (fields_autoplaced)
+    (property "Reference" "#PWR0108" (id 0) (at 123.19 107.95 0)
+      (effects (font (size 1.27 1.27)) hide)
+    )
+    (property "Value" "GNDPWR" (id 1) (at 123.063 107.95 0))
+    (property "Footprint" "" (id 2) (at 123.19 104.14 0)
+      (effects (font (size 1.27 1.27)) hide)
+    )
+    (property "Datasheet" "" (id 3) (at 123.19 104.14 0)
       (effects (font (size 1.27 1.27)) hide)
     )
@@
     (pin "9")
   )
+  (symbol (lib_id "power:GNDPWR") (at 135.89 139.7 0) (unit 1)
+    (in_bom yes) (on_board yes) (fields_autoplaced)
+    (property "Reference" "#PWR0107" (id 0) (at 135.89 144.78 0)
+      (effects (font (size 1.27 1.27)) hide)
+    )
+    (property "Value" "GNDPWR" (id 1) (at 135.763 144.78 0))
+    (property "Footprint" "" (id 2) (at 135.89 140.97 0)
+      (effects (font (size 1.27 1.27)) hide)
+    )
+    (property "Datasheet" "" (id 3) (at 135.89 140.97 0)
+      (effects (font (size 1.27 1.27)) hide)
+    )
+    (pin "1")
+  )
   (symbol (lib_id "Device:CP_Small") (at 143.51 54.61 0) (unit 1)
     (in_bom yes) (on_board yes)
@@
     (pin "2")
   )
+  (symbol (lib_id "power:GNDPWR") (at 123.19 139.7 0) (unit 1)
+    (in_bom yes) (on_board yes) (fields_autoplaced)
+    (property "Reference" "#PWR0106" (id 0) (at 123.19 144.78 0)
+      (effects (font (size 1.27 1.27)) hide)
+    )
+    (property "Value" "GNDPWR" (id 1) (at 123.063 144.78 0))
+    (property "Footprint" "" (id 2) (at 123.19 140.97 0)
+      (effects (font (size 1.27 1.27)) hide)
+    )
+    (property "Datasheet" "" (id 3) (at 123.19 140.97 0)
+      (effects (font (size 1.27 1.27)) hide)
+    )
+    (pin "1")
+  )
+  (symbol (lib_id "power:GNDPWR") (at 135.89 66.04 0) (unit 1)
+    (in_bom yes) (on_board yes) (fields_autoplaced)
+    (property "Reference" "#PWR0110" (id 0) (at 135.89 71.12 0)
+      (effects (font (size 1.27 1.27)) hide)
+    )
+    (property "Value" "GNDPWR" (id 1) (at 135.763 71.12 0))
+    (property "Footprint" "" (id 2) (at 135.89 67.31 0)
+      (effects (font (size 1.27 1.27)) hide)
+    )
+    (property "Datasheet" "" (id 3) (at 135.89 67.31 0)
+      (effects (font (size 1.27 1.27)) hide)
+    )
+    (pin "1")
+  )
 )

Commit message: 更新V3线路板
Parts:
- J6, J7, J8: value MOTOR -> PH2.0_1x06
Changed lines of the file:
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@@
       (effects (font (size 1.27 1.27)) (justify left))
     )
-    (property "Value" "MOTOR" (at 196.2912 128.651 0)
+    (property "Value" "PH2.0_1x06" (at 196.2912 128.651 0)
       (effects (font (size 1.27 1.27)) (justify left))
     )
@@
       (effects (font (size 1.27 1.27)) (justify left))
     )
-    (property "Value" "MOTOR" (at 196.2912 91.821 0)
+    (property "Value" "PH2.0_1x06" (at 196.2912 91.821 0)
       (effects (font (size 1.27 1.27)) (justify left))
     )
@@
       (effects (font (size 1.27 1.27)) (justify left))
     )
-    (property "Value" "MOTOR" (at 196.2912 56.261 0)
+    (property "Value" "PH2.0_1x06" (at 196.2912 56.261 0)
       (effects (font (size 1.27 1.27)) (justify left))
     )

Commit message: 添加v3初版设计
Parts:
- renumbered J6 to J7, J7 to J8, J8 to J9, U2 to U3, U3 to U4, U4 to U5

Commit message: 修改部分封装和值
Parts:
- C10, C11, C9: footprint Capacitor_SMD:CP_Elec_4x5.4 -> Capacitor_SMD:CP_Elec_5x5.4
Changed lines of the file:
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@@
       (effects (font (size 1.27 1.27)) (justify left))
     )
-    (property "Footprint" "Capacitor_SMD:CP_Elec_4x5.4" (at 143.51 128.27 0)
+    (property "Footprint" "Capacitor_SMD:CP_Elec_5x5.4" (at 143.51 128.27 0)
       (effects (font (size 1.27 1.27)) hide)
     )
@@
       (effects (font (size 1.27 1.27)) (justify left))
     )
-    (property "Footprint" "Capacitor_SMD:CP_Elec_4x5.4" (at 143.51 91.44 0)
+    (property "Footprint" "Capacitor_SMD:CP_Elec_5x5.4" (at 143.51 91.44 0)
       (effects (font (size 1.27 1.27)) hide)
     )
@@
       (effects (font (size 1.27 1.27)) (justify left))
     )
-    (property "Footprint" "Capacitor_SMD:CP_Elec_4x5.4" (at 143.51 54.61 0)
-      (effects (font (size 1.27 1.27)) hide)
-    )
+    (property "Footprint" "Capacitor_SMD:CP_Elec_5x5.4" (at 143.51 54.61 0)
+      (effects (font (size 1.27 1.27)) hide)
+    )
